File: PowerFullLamp_elec/PowerFullLamp_elec.kicad_sch (KiCad schematic)
At the start: 50 parts

Commit message: WIP trouver self
Parts:
- added C?: 22uf, Capacitor_SMD:C_1206_3216Metric_Pad1.33x1.80mm_HandSolder, symbol Device:C
- added C?: C, symbol Device:C
- added IC?: AP3429AKTTR-G1, samacsys:SOT95P280X100-5N, symbol samacsys:AP3429AKTTR-G1
- added L?: L, symbol Device:L
- added R?: 450k, Resistor_SMD:R_0805_2012Metric, symbol Device:R
- added R?: 100k, Resistor_SMD:R_0805_2012Metric, symbol Device:R
Connections:
- net +3V3: now also C?.1, IC?.1 (EN), IC?.3 (LX), L?.1
- net GND: now also C?.2, IC?.2 (GND), R?.1
- new net: C?.2, IC?.5 (FB), R?.1, R?.2
- new net: C?.1, L?.2, R?.2

Commit message: WIP routage
Parts:
- removed C?: C, symbol Device:C
- added C2: 22uf, Capacitor_SMD:C_1206_3216Metric_Pad1.33x1.80mm_HandSolder, symbol Device:C
- added TP1: Vin, TestPoint:TestPoint_THTPad_4.0x4.0mm_Drill2.0mm, symbol Connector:TestPoint
- added TP2: GND, TestPoint:TestPoint_THTPad_4.0x4.0mm_Drill2.0mm, symbol Connector:TestPoint
- L1: renamed from L?; value L -> 2u2H; footprint (none) -> Inductor_SMD:L_Wuerth_MAPI-3020
- gave numbers to parts that had none: 29
Connections:
- net +3V3: now also R1.2; no longer IC1.3 (LX)
- net GND: now also C2.2, TP2.1
- net at IC1.4 (VIN): now also C2.1, TP1.1
- net at L1.2: now also IC1.3 (LX); no longer R1.2
Other:
- moved on the sheet: L1
